File: isa-video/bus_interface.kicad_sch (KiCad schematic)
At the start: 11 parts, among them J5 Conn_ISA_8bit, U11 74HCT125, U4 74ALVC164245, U5 74ALVC164245

Commit message: V2.4 changes (#3)
Parts:
- gave numbers to parts that had none: 4
Changed lines of the file:
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@@
   (title_block
     (title "ISA Bus Interface")
-    (date "2023-09-17")
-    (rev "2.2")
+    (date "2024-01-04")
+    (rev "2.4")
   )
   (junction (at 149.86 168.91) (diameter 0) (color 0 0 0 0)
@@
           (reference "J5") (unit 1)
         )
-        (path "/de1f3d0f-5e30-4cf9-a891-fb3b803f4ea1"
-          (reference "J5") (unit 1)
-        )
       )
     )
@@
           (reference "U11") (unit 3)
         )
-        (path "/de1f3d0f-5e30-4cf9-a891-fb3b803f4ea1"
-          (reference "U?") (unit 3)
-        )
       )
     )
@@
           (reference "U11") (unit 4)
         )
-        (path "/de1f3d0f-5e30-4cf9-a891-fb3b803f4ea1"
-          (reference "U?") (unit 4)
-        )
       )
     )
@@
   (symbol (lib_id "Device:C_Small") (at 59.69 154.94 0) (unit 1)
     (in_bom yes) (on_board yes) (dnp no)
-    (property "Reference" "C?" (at 62.0268 153.7716 0)
+    (property "Reference" "C23" (at 62.0268 153.7716 0)
       (effects (font (size 1.27 1.27)) (justify left))
     )
@@
     (instances
       (project "isavideo"
-        (path "/de1f3d0f-5e30-4cf9-a891-fb3b803f4ea1/00000000-0000-0000-0000-00006043556f"
-          (reference "C?") (unit 1)
-        )
-        (path "/de1f3d0f-5e30-4cf9-a891-fb3b803f4ea1"
-          (reference "C?") (unit 1)
-        )
         (path "/de1f3d0f-5e30-4cf9-a891-fb3b803f4ea1/00000000-0000-0000-0000-00005fffc5de"
           (reference "C23") (unit 1)
@@
   (symbol (lib_id "Device:C_Small") (at 68.58 154.94 0) (unit 1)
     (in_bom yes) (on_board yes) (dnp no)
-    (property "Reference" "C?" (at 70.9168 153.7716 0)
+    (property "Reference" "C24" (at 70.9168 153.7716 0)
       (effects (font (size 1.27 1.27)) (justify left))
     )
@@
     (instances
       (project "isavideo"
-        (path "/de1f3d0f-5e30-4cf9-a891-fb3b803f4ea1/00000000-0000-0000-0000-00006043556f"
-          (reference "C?") (unit 1)
-        )
-        (path "/de1f3d0f-5e30-4cf9-a891-fb3b803f4ea1"
-          (reference "C?") (unit 1)
-        )
         (path "/de1f3d0f-5e30-4cf9-a891-fb3b803f4ea1/00000000-0000-0000-0000-00005fffc5de"
           (reference "C24") (unit 1)
@@
   (symbol (lib_id "power:+3V3") (at 59.69 148.59 0) (unit 1)
     (in_bom yes) (on_board yes) (dnp no)
-    (property "Reference" "#PWR?" (at 59.69 152.4 0)
+    (property "Reference" "#PWR066" (at 59.69 152.4 0)
       (effects (font (size 1.27 1.27)) hide)
     )
@@
     (instances
       (project "isavideo"
-        (path "/de1f3d0f-5e30-4cf9-a891-fb3b803f4ea1/00000000-0000-0000-0000-0000603a03ff"
-          (reference "#PWR?") (unit 1)
-        )
-        (path "/de1f3d0f-5e30-4cf9-a891-fb3b803f4ea1"
-          (reference "#PWR?") (unit 1)
-        )
         (path "/de1f3d0f-5e30-4cf9-a891-fb3b803f4ea1/00000000-0000-0000-0000-00005fffc5de"
           (reference "#PWR066") (unit 1)
@@
   (symbol (lib_id "power:GND") (at 68.58 161.29 0) (unit 1)
     (in_bom yes) (on_board yes) (dnp no)
-    (property "Reference" "#PWR?" (at 68.58 167.64 0)
+    (property "Reference" "#PWR068" (at 68.58 167.64 0)
       (effects (font (size 1.27 1.27)) hide)
     )
@@
     (instances
       (project "isavideo"
-        (path "/de1f3d0f-5e30-4cf9-a891-fb3b803f4ea1/00000000-0000-0000-0000-0000603a03ff"
-          (reference "#PWR?") (unit 1)
-        )
-        (path "/de1f3d0f-5e30-4cf9-a891-fb3b803f4ea1"
-          (reference "#PWR?") (unit 1)
-        )
         (path "/de1f3d0f-5e30-4cf9-a891-fb3b803f4ea1/00000000-0000-0000-0000-00005fffc5de"
           (reference "#PWR068") (unit 1)
@@
           (reference "#PWR067") (unit 1)
         )
-        (path "/de1f3d0f-5e30-4cf9-a891-fb3b803f4ea1"
-          (reference "#PWR?") (unit 1)
-        )
       )
     )
@@
   (symbol (lib_id "Device:C_Small") (at 77.47 154.94 0) (unit 1)
     (in_bom yes) (on_board yes) (dnp no)
-    (property "Reference" "C?" (at 79.8068 153.7716 0)
+    (property "Reference" "C25" (at 79.8068 153.7716 0)
       (effects (font (size 1.27 1.27)) (justify left))
     )
@@
     (instances
       (project "isavideo"
-        (path "/de1f3d0f-5e30-4cf9-a891-fb3b803f4ea1/00000000-0000-0000-0000-00006043556f"
-          (reference "C?") (unit 1)
-        )
-        (path "/de1f3d0f-5e30-4cf9-a891-fb3b803f4ea1"
-          (reference "C?") (unit 1)
-        )
         (path "/de1f3d0f-5e30-4cf9-a891-fb3b803f4ea1/00000000-0000-0000-0000-00005fffc5de"
           (reference "C25") (unit 1)
@@
   (symbol (lib_id "Device:C_Small") (at 86.36 154.94 0) (unit 1)
     (in_bom yes) (on_board yes) (dnp no)
-    (property "Reference" "C?" (at 88.6968 153.7716 0)
+    (property "Reference" "C26" (at 88.6968 153.7716 0)
       (effects (font (size 1.27 1.27)) (justify left))
     )
@@
     (instances
       (project "isavideo"
-        (path "/de1f3d0f-5e30-4cf9-a891-fb3b803f4ea1/00000000-0000-0000-0000-00006043556f"
-          (reference "C?") (unit 1)
-        )
-        (path "/de1f3d0f-5e30-4cf9-a891-fb3b803f4ea1"
-          (reference "C?") (unit 1)
-        )
         (path "/de1f3d0f-5e30-4cf9-a891-fb3b803f4ea1/00000000-0000-0000-0000-00005fffc5de"
           (reference "C26") (unit 1)
@@
   (symbol (lib_id "power:+3V3") (at 77.47 148.59 0) (unit 1)
     (in_bom yes) (on_board yes) (dnp no)
-    (property "Reference" "#PWR?" (at 77.47 152.4 0)
+    (property "Reference" "#PWR069" (at 77.47 152.4 0)
       (effects (font (size 1.27 1.27)) hide)
     )
@@
     (instances
       (project "isavideo"
-        (path "/de1f3d0f-5e30-4cf9-a891-fb3b803f4ea1/00000000-0000-0000-0000-0000603a03ff"
-          (reference "#PWR?") (unit 1)
-        )
-        (path "/de1f3d0f-5e30-4cf9-a891-fb3b803f4ea1"
-          (reference "#PWR?") (unit 1)
-        )
         (path "/de1f3d0f-5e30-4cf9-a891-fb3b803f4ea1/00000000-0000-0000-0000-00005fffc5de"
           (reference "#PWR069") (unit 1)
@@
   (symbol (lib_id "power:GND") (at 86.36 161.29 0) (unit 1)
     (in_bom yes) (on_board yes) (dnp no)
-    (property "Reference" "#PWR?" (at 86.36 167.64 0)
+    (property "Reference" "#PWR071" (at 86.36 167.64 0)
       (effects (font (size 1.27 1.27)) hide)
     )
@@
     (instances
       (project "isavideo"
-        (path "/de1f3d0f-5e30-4cf9-a891-fb3b803f4ea1/00000000-0000-0000-0000-0000603a03ff"
-          (reference "#PWR?") (unit 1)
-        )
-        (path "/de1f3d0f-5e30-4cf9-a891-fb3b803f4ea1"
-          (reference "#PWR?") (unit 1)
-        )
         (path "/de1f3d0f-5e30-4cf9-a891-fb3b803f4ea1/00000000-0000-0000-0000-00005fffc5de"
           (reference "#PWR071") (unit 1)
@@
           (reference "#PWR070") (unit 1)
         )
-        (path "/de1f3d0f-5e30-4cf9-a891-fb3b803f4ea1"
-          (reference "#PWR?") (unit 1)
-        )
-      )
+      )
