File: isa-video/isavideo.kicad_sch (KiCad schematic)
At the start: 37 parts, among them J1 PROG, J2 DB15_Female_HighDensity_Mount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, J3 PJRAN1X1U04X, J6 RFMOD, SW1 SW_DIP_x04, U1 ICE40HX4K-TQ144, U11 74HCT125, U2 SST26VF080A-104I/SN, U3 74ALVC164245, X1 10MHz, X2 14.318MHz

Commit message: V2.4 changes (#3)
Parts:
- gave numbers to parts that had none: 6
Connections:
- no-connect marks 25 -> 26
Changed lines of the file:
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@@
   (title_block
     (title "Top Level")
-    (date "2023-10-13")
-    (rev "2.3")
+    (date "2024-01-04")
+    (rev "2.4")
   )
   (junction (at 148.59 43.18) (diameter 0) (color 0 0 0 0)
@@
   (no_connect (at 191.77 130.81))
   (no_connect (at 227.33 133.35))
+  (no_connect (at 270.51 74.93))
   (no_connect (at 227.33 130.81))
   (no_connect (at 269.24 26.67))
@@
   (symbol (lib_id "Device:C_Small") (at 156.21 52.07 0) (unit 1)
     (in_bom yes) (on_board yes) (dnp no)
-    (property "Reference" "C?" (at 158.5468 50.9016 0)
+    (property "Reference" "C1" (at 158.5468 50.9016 0)
       (effects (font (size 1.27 1.27)) (justify left))
     )
@@
     (instances
       (project "isavideo"
-        (path "/de1f3d0f-5e30-4cf9-a891-fb3b803f4ea1/00000000-0000-0000-0000-00006043556f"
-          (reference "C?") (unit 1)
-        )
         (path "/de1f3d0f-5e30-4cf9-a891-fb3b803f4ea1"
           (reference "C1") (unit 1)
@@
   (symbol (lib_id "Device:C_Small") (at 161.29 144.78 0) (unit 1)
     (in_bom yes) (on_board yes) (dnp no)
-    (property "Reference" "C?" (at 163.6268 143.6116 0)
+    (property "Reference" "C30" (at 163.6268 143.6116 0)
       (effects (font (size 1.27 1.27)) (justify left))
     )
@@
     (instances
       (project "isavideo"
-        (path "/de1f3d0f-5e30-4cf9-a891-fb3b803f4ea1/00000000-0000-0000-0000-00006043556f"
-          (reference "C?") (unit 1)
-        )
         (path "/de1f3d0f-5e30-4cf9-a891-fb3b803f4ea1"
           (reference "C30") (unit 1)
@@
   (symbol (lib_id "Device:C_Small") (at 93.98 142.24 0) (unit 1)
     (in_bom yes) (on_board yes) (dnp no)
-    (property "Reference" "C?" (at 96.3168 141.0716 0)
+    (property "Reference" "C31" (at 96.3168 141.0716 0)
       (effects (font (size 1.27 1.27)) (justify left))
     )
@@
     (instances
       (project "isavideo"
-        (path "/de1f3d0f-5e30-4cf9-a891-fb3b803f4ea1/00000000-0000-0000-0000-00006043556f"
-          (reference "C?") (unit 1)
-        )
         (path "/de1f3d0f-5e30-4cf9-a891-fb3b803f4ea1"
           (reference "C31") (unit 1)
@@
   (symbol (lib_id "Device:C_Small") (at 254 151.13 0) (unit 1)
     (in_bom yes) (on_board yes) (dnp no)
-    (property "Reference" "C?" (at 256.3368 149.9616 0)
+    (property "Reference" "C21" (at 256.3368 149.9616 0)
       (effects (font (size 1.27 1.27)) (justify left))
     )
@@
     (instances
       (project "isavideo"
-        (path "/de1f3d0f-5e30-4cf9-a891-fb3b803f4ea1/00000000-0000-0000-0000-00006043556f"
-          (reference "C?") (unit 1)
-        )
         (path "/de1f3d0f-5e30-4cf9-a891-fb3b803f4ea1"
           (reference "C21") (unit 1)
@@
   (symbol (lib_id "Device:C_Small") (at 262.89 151.13 0) (unit 1)
     (in_bom yes) (on_board yes) (dnp no)
-    (property "Reference" "C?" (at 265.2268 149.9616 0)
+    (property "Reference" "C22" (at 265.2268 149.9616 0)
       (effects (font (size 1.27 1.27)) (justify left))
     )
@@
     (instances
       (project "isavideo"
-        (path "/de1f3d0f-5e30-4cf9-a891-fb3b803f4ea1/00000000-0000-0000-0000-00006043556f"
-          (reference "C?") (unit 1)
-        )
         (path "/de1f3d0f-5e30-4cf9-a891-fb3b803f4ea1"
           (reference "C22") (unit 1)
@@
   (symbol (lib_id "power:+3V3") (at 254 144.78 0) (unit 1)
     (in_bom yes) (on_board yes) (dnp no)
-    (property "Reference" "#PWR?" (at 254 148.59 0)
+    (property "Reference" "#PWR063" (at 254 148.59 0)
       (effects (font (size 1.27 1.27)) hide)
     )
@@
     (instances
       (project "isavideo"
-        (path "/de1f3d0f-5e30-4cf9-a891-fb3b803f4ea1/00000000-0000-0000-0000-0000603a03ff"
-          (reference "#PWR?") (unit 1)
-        )
         (path "/de1f3d0f-5e30-4cf9-a891-fb3b803f4ea1"
           (reference "#PWR063") (unit 1)
@@
   (symbol (lib_id "power:GND") (at 262.89 157.48 0) (unit 1)
     (in_bom yes) (on_board yes) (dnp no)
-    (property "Reference" "#PWR?" (at 262.89 163.83 0)
+    (property "Reference" "#PWR065" (at 262.89 163.83 0)
       (effects (font (size 1.27 1.27)) hide)
     )
@@
     (instances
       (project "isavideo"
-        (path "/de1f3d0f-5e30-4cf9-a891-fb3b803f4ea1/00000000-0000-0000-0000-0000603a03ff"
-          (reference "#PWR?") (unit 1)
-        )
         (path "/de1f3d0f-5e30-4cf9-a891-fb3b803f4ea1"
           (reference "#PWR065") (unit 1)
@@
   (symbol (lib_id "Device:C_Small") (at 153.67 97.79 0) (unit 1)
     (in_bom yes) (on_board yes) (dnp no)
-    (property "Reference" "C?" (at 156.0068 96.6216 0)
+    (property "Reference" "C20" (at 156.0068 96.6216 0)
       (effects (font (size 1.27 1.27)) (justify left))
     )
@@
     (instances
       (project "isavideo"
-        (path "/de1f3d0f-5e30-4cf9-a891-fb3b803f4ea1/00000000-0000-0000-0000-00006043556f"
-          (reference "C?") (unit 1)
-        )
         (path "/de1f3d0f-5e30-4cf9-a891-fb3b803f4ea1"
           (reference "C20") (unit 1)
