File: isa-video/vga_dac.kicad_sch (KiCad schematic)
At the start: 20 parts, among them U6 ADA4891-3

Commit message: V2.4 changes (#3)
Parts:
- gave numbers to parts that had none: 1
Connections:
- no-connect marks 0 -> 4
Changed lines of the file:
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@@
   (title_block
     (title "Resistor Ladder DAC and Output Buffer")
-    (date "2023-09-17")
-    (rev "2.2")
+    (date "2024-01-04")
+    (rev "2.4")
   )
   (junction (at 116.84 130.81) (diameter 0) (color 0 0 0 0)
@@
   (junction (at 115.57 173.99) (diameter 0) (color 0 0 0 0)
   )
+  (no_connect (at 130.81 135.89))
+  (no_connect (at 130.81 133.35))
+  (no_connect (at 120.65 135.89))
+  (no_connect (at 120.65 133.35))
   (bus_entry (at 100.33 59.69) (size 2.54 2.54)
     (stroke (width 0) (type default))
@@
           (reference "U6") (unit 1)
         )
-        (path "/de1f3d0f-5e30-4cf9-a891-fb3b803f4ea1"
-          (reference "U?") (unit 1)
-        )
       )
     )
@@
           (reference "U6") (unit 2)
         )
-        (path "/de1f3d0f-5e30-4cf9-a891-fb3b803f4ea1"
-          (reference "U?") (unit 2)
-        )
       )
     )
@@
           (reference "U6") (unit 3)
         )
-        (path "/de1f3d0f-5e30-4cf9-a891-fb3b803f4ea1"
-          (reference "U?") (unit 3)
-        )
       )
     )
@@
           (reference "U6") (unit 4)
         )
-        (path "/de1f3d0f-5e30-4cf9-a891-fb3b803f4ea1"
-          (reference "U?") (unit 4)
-        )
       )
     )
@@
           (reference "U6") (unit 5)
         )
-        (path "/de1f3d0f-5e30-4cf9-a891-fb3b803f4ea1"
-          (reference "U?") (unit 5)
-        )
       )
     )
@@
           (reference "RN1") (unit 1)
         )
-        (path "/de1f3d0f-5e30-4cf9-a891-fb3b803f4ea1"
-          (reference "RN?") (unit 1)
-        )
       )
     )
@@
           (reference "RN2") (unit 1)
         )
-        (path "/de1f3d0f-5e30-4cf9-a891-fb3b803f4ea1"
-          (reference "RN?") (unit 1)
-        )
       )
     )
@@
           (reference "RN7") (unit 1)
         )
-        (path "/de1f3d0f-5e30-4cf9-a891-fb3b803f4ea1"
-          (reference "RN?") (unit 1)
-        )
       )
     )
@@
           (reference "RN8") (unit 1)
         )
-        (path "/de1f3d0f-5e30-4cf9-a891-fb3b803f4ea1"
-          (reference "RN?") (unit 1)
-        )
       )
     )
@@
           (reference "RN9") (unit 1)
         )
-        (path "/de1f3d0f-5e30-4cf9-a891-fb3b803f4ea1"
-          (reference "RN?") (unit 1)
-        )
       )
     )
@@
           (reference "RN3") (unit 1)
         )
-        (path "/de1f3d0f-5e30-4cf9-a891-fb3b803f4ea1"
-          (reference "RN?") (unit 1)
-        )
       )
     )
@@
           (reference "RN4") (unit 1)
         )
-        (path "/de1f3d0f-5e30-4cf9-a891-fb3b803f4ea1"
-          (reference "RN?") (unit 1)
-        )
       )
     )
@@
           (reference "RN10") (unit 1)
         )
-        (path "/de1f3d0f-5e30-4cf9-a891-fb3b803f4ea1"
-          (reference "RN?") (unit 1)
-        )
       )
     )
@@
           (reference "RN5") (unit 1)
         )
-        (path "/de1f3d0f-5e30-4cf9-a891-fb3b803f4ea1"
-          (reference "RN?") (unit 1)
-        )
       )
     )
@@
           (reference "RN6") (unit 1)
         )
-        (path "/de1f3d0f-5e30-4cf9-a891-fb3b803f4ea1"
-          (reference "RN?") (unit 1)
-        )
       )
     )
@@
   (symbol (lib_id "Device:C_Small") (at 180.34 129.54 0) (unit 1)
     (in_bom yes) (on_board yes) (dnp no)
-    (property "Reference" "C?" (at 182.6768 128.3716 0)
+    (property "Reference" "C27" (at 182.6768 128.3716 0)
       (effects (font (size 1.27 1.27)) (justify left))
     )
@@
     (instances
       (project "isavideo"
-        (path "/de1f3d0f-5e30-4cf9-a891-fb3b803f4ea1/00000000-0000-0000-0000-00006043556f"
-          (reference "C?") (unit 1)
-        )
-        (path "/de1f3d0f-5e30-4cf9-a891-fb3b803f4ea1"
-          (reference "C?") (unit 1)
-        )
         (path "/de1f3d0f-5e30-4cf9-a891-fb3b803f4ea1/00000000-0000-0000-0000-0000601ac602"
           (reference "C27") (unit 1)
@@
   (symbol (lib_id "power:GND") (at 180.34 135.89 0) (unit 1)
     (in_bom yes) (on_board yes) (dnp no)
-    (property "Reference" "#PWR?" (at 180.34 142.24 0)
+    (property "Reference" "#PWR073" (at 180.34 142.24 0)
       (effects (font (size 1.27 1.27)) hide)
     )
@@
     (instances
       (project "isavideo"
-        (path "/de1f3d0f-5e30-4cf9-a891-fb3b803f4ea1/00000000-0000-0000-0000-0000603a03ff"
-          (reference "#PWR?") (unit 1)
-        )
-        (path "/de1f3d0f-5e30-4cf9-a891-fb3b803f4ea1"
-          (reference "#PWR?") (unit 1)
-        )
         (path "/de1f3d0f-5e30-4cf9-a891-fb3b803f4ea1/00000000-0000-0000-0000-0000601ac602"
           (reference "#PWR073") (unit 1)
